File: pcb/spektro-badge.kicad_sch (KiCad schematic)
At the start: 0 parts

Commit message: updating the project with new schematics, still unfinished
Parts:
- added C1, C2, C3: 100n, symbol Device:C
- added C4: 4.7u, Capacitor_SMD:C_0603_1608Metric, symbol Device:C
- added C5: 10n, Capacitor_SMD:C_0603_1608Metric, symbol Device:C
- added C6: 1u, Capacitor_SMD:C_0603_1608Metric, symbol Device:C
- added U1: STM32F030C8Tx, Package_QFP:LQFP-48_7x7mm_P0.5mm, symbol MCU_ST_STM32F0:STM32F030C8Tx
Connections:
- new net +3V3: C1.1, C2.1, C3.1, C4.1, C5.1, C6.1, U1.1 (VDD), U1.24 (VDD), U1.48 (VDD), U1.9 (VDDA)
- new net GND: C1.2, C2.2, C3.2, C4.2, C5.2, C6.2, U1.23 (VSS), U1.47 (VSS), U1.8 (VSSA)
Other:
- added sheet LED grid (grid.kicad_sch)
- added sheet Power (power.kicad_sch)
